File: Electrical/KiCad/BasePCB/BasePCB.kicad_sch (KiCad schematic)
At the start: 17 parts, among them J1 Conn_01x02_Socket, J10 Conn_01x08, J2 Conn_01x02_Socket, J3 Conn_01x06_Socket, J4 Conn_01x06_Socket, J5 Conn_01x06, J6 Conn_01x03, J7 Conn_01x03, J8 Conn_01x04, J9 Conn_01x08, Q1 AO3400A, Q2 AO3400A

Commit message: Add the base PCB gerbers and JLCPCB production files
Parts:
- removed A1: RaspberryPi_Pico, Module:RaspberryPi_Pico_SMD, symbol MCU_Module:RaspberryPi_Pico_Extensive
- added A2: RaspberryPi_Pico_W, Module:RaspberryPi_Pico_W_SMD, symbol MCU_Module:RaspberryPi_Pico_W_Extensive
- R3: value 570k -> 100k
- R4: value 330k -> 56k
Connections:
- net +3.3V: now also A2.36 (3V3)
- net +5V: now also A2.39 (VSYS)
- net +BATT: no longer J10.2 (Pin_2)
- net 5V_EN: now also A2.29 (GPIO22)
- net AIN1: now also A2.6 (GPIO4); no longer J9.6 (Pin_6)
- net AIN2: now also A2.7 (GPIO5); no longer J9.5 (Pin_5)
- net BIN1: now also A2.10 (GPIO7); no longer J9.3 (Pin_3)
- net BIN2: now also A2.9 (GPIO6); no longer J9.4 (Pin_4)
- net CLK: now also A2.24 (GPIO18)
- net CS: now also A2.27 (GPIO21)
- net EA1: now also A2.17 (GPIO13)
- net EA2: now also A2.16 (GPIO12)
- net EB1: now also A2.4 (GPIO2)
- net EB2: now also A2.5 (GPIO3)
- net GND: now also A2.13 (GND), A2.18 (GND), A2.23 (GND), A2.28 (GND), A2.3 (GND), A2.38 (GND), A2.8 (GND), A2.D2 (GND); no longer J10.1 (Pin_1), J9.1 (Pin_1)
- net MA1: now also J3.5 (Pin_5); no longer J10.6 (Pin_6), J3.6 (Pin_6)
- net MA2: now also J3.6 (Pin_6); no longer J10.5 (Pin_5), J3.5 (Pin_5)
- net MB1: now also J4.5 (Pin_5); no longer J10.3 (Pin_3), J4.6 (Pin_6)
- net MB2: now also J4.6 (Pin_6); no longer J10.4 (Pin_4), J4.5 (Pin_5)
- net MISO: now also A2.26 (GPIO20)
- net MOSI: now also A2.25 (GPIO19)
- net SA_PWM: now also A2.2 (GPIO1)
- net SA_PWR: now also A2.1 (GPIO0)
- net SB_PWM: now also A2.19 (GPIO14)
- net SB_PWR: now also A2.20 (GPIO15)
- net Vchg: now also A2.31 (GPIO26_ADC0)
- net nSLEEP: no longer J9.7 (Pin_7)
Other:
- moved on the sheet: J10, J9
